File: Main_PCB.kicad_sch (KiCad schematic)
At the start: 57 parts, among them IC1 TCN75AVUA713-VAO, IC2 24AA64T-I_OT, J1 Conn_Coaxial, J2 Conn_02x03_Odd_Even, J3 USB_C_Receptacle_USB2.0, J4 Conn_01x03_Male, J5 Conn_01x08, J6 Conn_01x08, SW1 SW_Push, SW2 SW_Push, U1 LTR-329ALS-01, U2 RFM95W-868S2, U3 1013, U4 STM32L476RGTx, U5 ATECC508A-SSHDA-T, U6 ST-Nucleo-L432KC, U7 USBLC6-2SC6, Y1 32.768

Commit message: updated b2b connector
Parts:
- J5: footprint Connector_JST:JST_EH_B8B-EH-A_1x08_P2.50mm_Vertical -> Connector_Molex:Molex_Micro-Latch_53253-0870_1x08_P2.00mm_Vertical
- J6: footprint Connector_JST:JST_EH_S8B-EH_1x08_P2.50mm_Horizontal -> Connector_Molex:Molex_Micro-Latch_53253-0870_1x08_P2.00mm_Vertical
Changed lines of the file:
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@@
       (effects (font (size 1.27 1.27)) (justify left))
     )
-    (property "Footprint" "Connector_JST:JST_EH_B8B-EH-A_1x08_P2.50mm_Vertical" (id 2) (at 334.01 153.67 0)
+    (property "Footprint" "Connector_Molex:Molex_Micro-Latch_53253-0870_1x08_P2.00mm_Vertical" (id 2) (at 334.01 153.67 0)
       (effects (font (size 1.27 1.27)) hide)
     )
@@
     (property "Reference" "J6" (id 0) (at 346.0115 139.7 0))
     (property "Value" "Conn_01x08" (id 1) (at 346.0115 142.24 0))
-    (property "Footprint" "Connector_JST:JST_EH_S8B-EH_1x08_P2.50mm_Horizontal" (id 2) (at 344.17 156.21 0)
+    (property "Footprint" "Connector_Molex:Molex_Micro-Latch_53253-0870_1x08_P2.00mm_Vertical" (id 2) (at 344.17 156.21 0)
       (effects (font (size 1.27 1.27)) hide)
     )
@@
     )
     (path "/cb3aca7e-8766-46d7-af6a-1e4b8da68729"
-      (reference "J5") (unit 1) (value "Conn_01x08") (footprint "Connector_JST:JST_EH_B8B-EH-A_1x08_P2.50mm_Vertical")
+      (reference "J5") (unit 1) (value "Conn_01x08") (footprint "Connector_Molex:Molex_Micro-Latch_53253-0870_1x08_P2.00mm_Vertical")
     )
     (path "/4c2589f5-6376-48ce-98db-462c0484826b"
-      (reference "J6") (unit 1) (value "Conn_01x08") (footprint "Connector_JST:JST_EH_S8B-EH_1x08_P2.50mm_Horizontal")
+      (reference "J6") (unit 1) (value "Conn_01x08") (footprint "Connector_Molex:Molex_Micro-Latch_53253-0870_1x08_P2.00mm_Vertical")
     )
     (path "/c75b443c-d4e7-4644-a8d9-c7a2ddb573ca"
